File: clock/clock.kicad_pcb (KiCad board)
At the start: 2 copper layers, 176.8 x 81.3 mm, 295 parts, among them P101 CONN_01X03, P102 CONN_FAN_PWM, P103 XG4A-1631, P301 MCRF, P401 CONN_01X10, Q201 MMBT3904, U201 PCA9306, U202 DAC8830, U203 LMV722, U204 LTC2990, U205 LP3853, U207 NC7SZ125, U301 Adafruit746, U302 MIC5225, U303 PA6H, U401 74LVC541, U501 TPS56428, U502 TPS56428, U503 TPS56428, U601 ADT7410, U602 DS3231, U603 ADT7410, Y202 CX210

Commit message: More clean up...
Parts:
- removed the REF** at (334.0, 196.6)
- removed the REF** at (317.0, 201.7)
- removed the REF** at (312.9, 201.7)
- removed the REF** at (316.1, 208.3)
- removed the REF** at (324.9, 202.4)
- removed the REF** at (283.2, 195.1)
- removed the REF** at (248.9, 213.4)
- added REF**: Stitching_Via_40x24mil, local:Stitching_Via_40x24mil, F.Cu at (322.6, 201.7)
- added REF**: Stitching_Via_40x24mil, local:Stitching_Via_40x24mil, F.Cu at (241.3, 201.2)
- added REF**: Stitching_Via_40x24mil, local:Stitching_Via_40x24mil, F.Cu at (238.8, 201.2)
- added REF**: Stitching_Via_40x24mil, local:Stitching_Via_40x24mil, F.Cu at (236.2, 201.2)
- added REF**: Stitching_Via_40x24mil, local:Stitching_Via_40x24mil, F.Cu at (248.9, 201.2)
- added REF**: Stitching_Via_40x24mil, local:Stitching_Via_40x24mil, F.Cu at (320.0, 201.7)
- added REF**: Stitching_Via_40x24mil, local:Stitching_Via_40x24mil, F.Cu at (312.4, 201.7)
- added REF**: Stitching_Via_40x24mil, local:Stitching_Via_40x24mil, F.Cu at (363.2, 208.3)
- added REF**: Stitching_Via_40x24mil, local:Stitching_Via_40x24mil, F.Cu at (255.3, 230.6)
- added REF**: Stitching_Via_40x24mil, local:Stitching_Via_40x24mil, F.Cu at (332.7, 243.8)
- added REF**: Stitching_Via_40x24mil, local:Stitching_Via_40x24mil, F.Cu at (299.7, 243.8)
- added REF**: Stitching_Via_40x24mil, local:Stitching_Via_40x24mil, F.Cu at (339.1, 206.8)
- added REF**: Stitching_Via_40x24mil, local:Stitching_Via_40x24mil, F.Cu at (336.6, 206.8)
- moved REF** 9.23 mm to (266.7, 241.3)
- moved REF** 4.06 mm to (304.8, 201.7)
- moved REF** 3.56 mm to (307.3, 201.7)
- moved REF** 3.32 mm to (332.7, 205.7)
- moved REF** 2.54 mm to (358.1, 243.8)
- moved REF** 2.54 mm to (353.1, 243.8)
- moved REF** 2.40 mm to (348.0, 208.3)
- moved REF** 2.40 mm to (350.5, 208.3)
- moved REF** 2.34 mm to (353.1, 218.4)
- moved REF** 1.98 mm to (271.8, 236.2)
- moved REF** 1.98 mm to (274.3, 236.2)
- moved REF** 1.98 mm to (276.9, 236.2)
- moved REF** 1.98 mm to (276.9, 241.3)
- moved REF** 1.98 mm to (271.8, 241.3)
- moved REF** 1.93 mm to (261.6, 201.2)
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Routing:
- net /ocxo/SCL5: track 111.8 -> 128.0 mm
- net /power/+3.0V_PG: track 167.2 -> 158.8 mm, vias 5 -> 4
- net /microzed/+1.8V_PG: track 149.3 -> 143.2 mm, vias 9 -> 8
- net /microzed/RTC_SDA: track 43.2 -> 41.7 mm, vias 3 -> 2
- net /microzed/~DAC_CS~: track 36.2 -> 35.3 mm
- net /microzed/RTC_SCL: vias 3 -> 2

Commit message: Minor clean up. Regenerate gerbers.
Parts:
- removed the REF** at (214.9, 168.7)
- removed the REF** at (212.3, 168.7)
- removed the REF** at (209.8, 168.7)
- removed the REF** at (207.3, 168.7)
- added REF**: Stitching_Via_40x24mil, local:Stitching_Via_40x24mil, F.Cu at (233.7, 185.4)
- moved REF** 2.09 mm to (254.0, 218.4)
- moved REF** 1.48 mm to (205.7, 203.2)
- moved REF** 1.48 mm to (205.7, 198.1)
- moved REF** 1.48 mm to (205.7, 195.6)
- moved REF** 1.48 mm to (205.7, 193.0)
- moved REF** 1.48 mm to (198.1, 203.2)
- moved REF** 1.48 mm to (203.2, 203.2)
- moved REF** 0.80 mm to (198.1, 198.1)
- moved REF** 0.80 mm to (198.1, 195.6)
- moved REF** 0.80 mm to (198.1, 193.0)
- moved REF** 0.51 mm to (281.9, 212.1)
- moved REF** 0.25 mm to (281.9, 204.5)
- moved REF** 0.25 mm to (284.5, 204.5)
- moved REF** 0.25 mm to (279.4, 204.5)
Routing:
- net VIN: track 327.1 -> 328.0 mm

Commit message: Generate PDF schematics.
Other:
- board text added: "dcsun88osh@gmail.com"
- board text removed: "dcsun88@gmail.com"
Changed lines of the file:
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@@
     (effects (font (size 0.75 0.75) (thickness 0.15)))
   )
-  (gr_text dcsun88@gmail.com (at 241.3 166.37) (layer F.SilkS)
+  (gr_text dcsun88osh@gmail.com (at 241.3 166.37) (layer F.SilkS)
     (effects (font (size 0.75 0.75) (thickness 0.15)))
   )
