File: clock/rtctemp.sch (KiCad schematic (older format))
At the start: 19 parts, among them U601 ADT7410, U602 DS3231, U603 ADT7410

Commit message: Update clock board to kicad 5.1. Regenerate output files.
Parts:
- BT601: symbol Battery -> Local:Battery
- C601, C602, C603: symbol C -> Device:C
- R601, R602, R603, R604, R605, R606, R607, R608, R609, R610, R611, R612: symbol R_local -> Local:R_local
- U601, U603: symbol ADT7410 -> Local:ADT7410
- U602: symbol DS3231 -> Local:DS3231
Changed lines of the file:
@@
-EESchema Schematic File Version 2
-LIBS:clock-rescue
-LIBS:local
-LIBS:power
-LIBS:device
-LIBS:transistors
-LIBS:conn
-LIBS:linear
-LIBS:regul
-LIBS:74xx
-LIBS:cmos4000
-LIBS:adc-dac
-LIBS:memory
-LIBS:xilinx
-LIBS:microcontrollers
-LIBS:dsp
-LIBS:microchip
-LIBS:analog_switches
-LIBS:motorola
-LIBS:texas
-LIBS:intel
-LIBS:audio
-LIBS:interface
-LIBS:digital-audio
-LIBS:philips
-LIBS:display
-LIBS:cypress
-LIBS:siliconi
-LIBS:opto
-LIBS:atmel
-LIBS:contrib
-LIBS:valves
-LIBS:clock-cache
-EELAYER 25 0
+EESchema Schematic File Version 4
+EELAYER 30 0
 EELAYER END
 $Descr A4 11693 8268
@@
 $EndDescr
 $Comp
-L DS3231 U602
+L Local:DS3231 U602
 U 1 1 5636A7B6
 P 5750 2700
@@
 $EndComp
 $Comp
-L ADT7410 U601
+L Local:ADT7410 U601
 U 1 1 5636A81E
 P 4200 5050
@@
 	5750 3300 5750 3500
 $Comp
-L GND #PWR082
+L power:GND #PWR082
 U 1 1 5636B6C4
 P 5750 3500
@@
 $EndComp
 $Comp
-L VCC #PWR083
+L Local:VCC #PWR083
 U 1 1 5636B7D2
 P 5750 2000
@@
 	5750 2000 5750 2100
 $Comp
-L R_local R603
+L Local:R_local R603
 U 1 1 5636BA4F
 P 4050 2050
@@
 $EndComp
 $Comp
-L R_local R604
+L Local:R_local R604
 U 1 1 5636BAB4
 P 4500 2050
@@
 	4500 1800 4500 1900
 $Comp
-L VCC #PWR084
+L Local:VCC #PWR084
 U 1 1 5636BBAE
 P 4300 1700
@@
 $EndComp
 $Comp
-L Battery BT601
+L Local:Battery BT601
 U 1 1 5636BBED
 P 6950 2800
@@
 	6950 2550 6950 2650
 $Comp
-L GND #PWR085
+L power:GND #PWR085
 U 1 1 5636BC94
 P 6950 3050
@@
 Connection ~ 4500 2350
 $Comp
-L ADT7410 U603
+L Local:ADT7410 U603
 U 1 1 5636C07C
 P 9050 5050
@@
 $EndComp
 $Comp
-L VCC #PWR086
+L Local:VCC #PWR086
 U 1 1 5636C0D5
 P 4200 4450
@@
 	9050 5650 9050 5550
 $Comp
-L GND #PWR087
+L power:GND #PWR087
 U 1 1 5636C104
 P 9050 5650
@@
 	4200 5650 4200 5550
 $Comp
-L GND #PWR088
+L power:GND #PWR088
 U 1 1 5636C11B
 P 4200 5650
@@
 $EndComp
 $Comp
-L R_local R605
+L Local:R_local R605
 U 1 1 5636C195
 P 7500 4550
@@
 $EndComp
 $Comp
-L R_local R606
+L Local:R_local R606
 U 1 1 5636C19F
 P 7950 4550
@@
 	7950 4300 7950 4400
 $Comp
-L VCC #PWR089
+L Local:VCC #PWR089
 U 1 1 5636C1AA
 P 7750 4200
@@
 Connection ~ 7500 4950
 $Comp
-L R_local R601
+L Local:R_local R601
 U 1 1 5636C415
 P 3100 5600
@@
 $EndComp
 $Comp
-L R_local R602
+L Local:R_local R602
 U 1 1 5636C41F
 P 3550 5600
@@
 Connection ~ 3550 5850
 $Comp
-L GND #PWR090
+L power:GND #PWR090
 U 1 1 5636C550
 P 3550 5950
@@
 $EndComp
 $Comp
-L R_local R608
+L Local:R_local R608
 U 1 1 5636C5C2
 P 8400 5550
@@
 	8400 5250 8400 5400
 $Comp
-L GND #PWR091
+L power:GND #PWR091
 U 1 1 5636C5CD
 P 8400 5800
@@
 $EndComp
 $Comp
-L R_local R607
+L Local:R_local R607
 U 1 1 5636C65B
 P 8400 4550
@@
 Connection ~ 3500 4950
 $Comp
-L GND #PWR092
+L power:GND #PWR092
 U 1 1 5636CF30
 P 8550 2750
@@
 	8550 2350 8550 2250
 $Comp
-L C C603
+L Device:C C603
 U 1 1 5636CF43
 P 8550 2500
@@
 $EndComp
 $Comp
-L VCC #PWR093
+L Local:VCC #PWR093
 U 1 1 5636D2DE
 P 8550 2250
@@
 $EndComp
 $Comp
-L GND #PWR094
+L power:GND #PWR094
 U 1 1 5636D43C
 P 5600 5900
@@
 	5600 5500 5600 5400
 $Comp
-L C C601
+L Device:C C601
 U 1 1 5636D449
 P 5600 5650
@@
 $EndComp
 $Comp
-L VCC #PWR095
+L Local:VCC #PWR095
 U 1 1 5636D44F
 P 5600 5400
@@
 $EndComp
 $Comp
-L GND #PWR096
+L power:GND #PWR096
 U 1 1 5636D49F
 P 7750 6000
@@
 	7750 5600 7750 5500
 $Comp
-L C C602
+L Device:C C602
 U 1 1 5636D4AC
 P 7750 5750
@@
 $EndComp
 $Comp
-L VCC #PWR097
+L Local:VCC #PWR097
 U 1 1 5636D4B2
 P 7750 5500
@@
 NoConn ~ 5150 2550
 $Comp
-L VCC #PWR098
+L Local:VCC #PWR098
 U 1 1 563E1DA8
 P 9050 4450
@@
 	8400 5800 8400 5700
 $Comp
-L PWR_FLAG #FLG099
+L power:PWR_FLAG #FLG099
 U 1 1 564556C2
 P 7300 2450
@@
 Connection ~ 7300 2550
 $Comp
-L R_local R609
+L Local:R_local R609
 U 1 1 57AC1154
 P 6500 1450
@@
 $EndComp
 $Comp
-L R_local R610
+L Local:R_local R610
 U 1 1 57AC1181
 P 7050 1450
@@
 Connection ~ 6500 1700
 $Comp
-L VCC #PWR0100
+L Local:VCC #PWR0100
 U 1 1 57AC17FC
 P 7050 1100
@@
 i2c_addr = 0x49
 $Comp
-L R_local R612
+L Local:R_local R612
 U 1 1 589A8EE4
 P 9850 4550
@@
 $EndComp
 $Comp
-L VCC #PWR0101
+L Local:VCC #PWR0101
 U 1 1 589A8FE2
 P 9850 4300
@@
 	9850 4700 9850 4850
 $Comp
-L R_local R611
+L Local:R_local R611
 U 1 1 589A91FB
 P 5000 4550
@@
 $EndComp
 $Comp
-L VCC #PWR0102
+L Local:VCC #PWR0102
 U 1 1 589A9201
 P 5000 4300
