File: rj45brkout/rj45brkout.sch (KiCad schematic (older format))
At the start: 13 parts, among them J101 RJ45_LEDS, P101 CONN_01X01, P102 CONN_01X01, P103 CONN_01X01, P104 CONN_01X01, P105 CONN_01X01, P106 CONN_01X01, P107 CONN_01X01, P108 CONN_01X01, P109 CONN_01X01, P110 CONN_01X01, P111 CONN_01X01, P112 CONN_01X01

Commit message: Update rj45 break out board to kicad 5.1. Regenerate output files.
Parts:
- J101: symbol RJ45_LEDS -> Local:RJ45_LEDS
- P101, P102, P103, P104, P105, P106, P107, P108, P109, P110, P111, P112: symbol CONN_01X01 -> conn:CONN_01X01
Changed lines of the file:
@@
-EESchema Schematic File Version 2
-LIBS:local
-LIBS:power
-LIBS:device
-LIBS:transistors
-LIBS:conn
-LIBS:linear
-LIBS:regul
-LIBS:74xx
-LIBS:cmos4000
-LIBS:adc-dac
-LIBS:memory
-LIBS:xilinx
-LIBS:microcontrollers
-LIBS:dsp
-LIBS:microchip
-LIBS:analog_switches
-LIBS:motorola
-LIBS:texas
-LIBS:intel
-LIBS:audio
-LIBS:interface
-LIBS:digital-audio
-LIBS:philips
-LIBS:display
-LIBS:cypress
-LIBS:siliconi
-LIBS:opto
-LIBS:atmel
-LIBS:contrib
-LIBS:valves
-LIBS:rj45brkout-cache
-EELAYER 25 0
+EESchema Schematic File Version 4
+EELAYER 30 0
 EELAYER END
 $Descr A4 11693 8268
@@
 $EndDescr
 $Comp
-L RJ45_LEDS J101
+L Local:RJ45_LEDS J101
 U 1 1 5AD92762
 P 6400 3800
@@
 $EndComp
 $Comp
-L CONN_01X01 P107
+L conn:CONN_01X01 P107
 U 1 1 5AD927DD
 P 4950 3500
@@
 $EndComp
 $Comp
-L CONN_01X01 P108
+L conn:CONN_01X01 P108
 U 1 1 5AD928A6
 P 4950 3700
@@
 $EndComp
 $Comp
-L CONN_01X01 P106
+L conn:CONN_01X01 P106
 U 1 1 5AD928DB
 P 4950 3250
@@
 $EndComp
 $Comp
-L CONN_01X01 P105
+L conn:CONN_01X01 P105
 U 1 1 5AD9293F
 P 4950 3050
@@
 $EndComp
 $Comp
-L CONN_01X01 P109
+L conn:CONN_01X01 P109
 U 1 1 5AD92962
 P 5125 4300
@@
 $EndComp
 $Comp
-L CONN_01X01 P110
+L conn:CONN_01X01 P110
 U 1 1 5AD929A4
 P 5125 4500
@@
 $EndComp
 $Comp
-L CONN_01X01 P111
+L conn:CONN_01X01 P111
 U 1 1 5AD929DB
 P 6150 4700
@@
 $EndComp
 $Comp
-L CONN_01X01 P112
+L conn:CONN_01X01 P112
 U 1 1 5AD92A13
 P 6150 4900
@@
 $EndComp
 $Comp
-L CONN_01X01 P104
+L conn:CONN_01X01 P104
 U 1 1 5AD92A4C
 P 4950 2800
@@
 $EndComp
 $Comp
-L CONN_01X01 P103
+L conn:CONN_01X01 P103
 U 1 1 5AD92A90
 P 4950 2600
@@
 $EndComp
 $Comp
-L CONN_01X01 P102
+L conn:CONN_01X01 P102
 U 1 1 5AD92ACD
 P 4950 2350
@@
 $EndComp
 $Comp
-L CONN_01X01 P101
+L conn:CONN_01X01 P101
 U 1 1 5AD92B31
 P 4950 2150
@@
 $EndComp
 $Comp
-L GND #PWR01
+L power:GND #PWR01
 U 1 1 5AD92B85
 P 5675 4800

Commit message: Fix rj45 break out board to point to 5.1 symbol libraries. Fix USB-A break out board to point to 5.1 symbol libraries. Fix USB-B break out board to point to 5.1 symbol libraries.
Parts:
- P101, P102, P103, P104, P105, P106, P107, P108, P109, P110, P111, P112: symbol conn:CONN_01X01 -> Connector_Generic:Conn_01x01
Changed lines of the file:
@@
 $EndComp
 $Comp
-L conn:CONN_01X01 P107
+L Connector_Generic:Conn_01x01 P107
 U 1 1 5AD927DD
 P 4950 3500
@@
 $EndComp
 $Comp
-L conn:CONN_01X01 P108
+L Connector_Generic:Conn_01x01 P108
 U 1 1 5AD928A6
 P 4950 3700
@@
 $EndComp
 $Comp
-L conn:CONN_01X01 P106
+L Connector_Generic:Conn_01x01 P106
 U 1 1 5AD928DB
 P 4950 3250
@@
 $EndComp
 $Comp
-L conn:CONN_01X01 P105
+L Connector_Generic:Conn_01x01 P105
 U 1 1 5AD9293F
 P 4950 3050
@@
 $EndComp
 $Comp
-L conn:CONN_01X01 P109
+L Connector_Generic:Conn_01x01 P109
 U 1 1 5AD92962
 P 5125 4300
@@
 $EndComp
 $Comp
-L conn:CONN_01X01 P110
+L Connector_Generic:Conn_01x01 P110
 U 1 1 5AD929A4
 P 5125 4500
@@
 $EndComp
 $Comp
-L conn:CONN_01X01 P111
+L Connector_Generic:Conn_01x01 P111
 U 1 1 5AD929DB
 P 6150 4700
@@
 $EndComp
 $Comp
-L conn:CONN_01X01 P112
+L Connector_Generic:Conn_01x01 P112
 U 1 1 5AD92A13
 P 6150 4900
@@
 $EndComp
 $Comp
-L conn:CONN_01X01 P104
+L Connector_Generic:Conn_01x01 P104
 U 1 1 5AD92A4C
 P 4950 2800
@@
 $EndComp
 $Comp
-L conn:CONN_01X01 P103
+L Connector_Generic:Conn_01x01 P103
 U 1 1 5AD92A90
 P 4950 2600
@@
 $EndComp
 $Comp
-L conn:CONN_01X01 P102
+L Connector_Generic:Conn_01x01 P102
 U 1 1 5AD92ACD
 P 4950 2350
@@
 $EndComp
 $Comp
-L conn:CONN_01X01 P101
+L Connector_Generic:Conn_01x01 P101
 U 1 1 5AD92B31
 P 4950 2150
