File: usbabrkout/usbabrkout.sch (KiCad schematic (older format))
At the start: 6 parts, among them P101 CONN_01X01, P102 CONN_01X01, P103 CONN_01X01, P104 CONN_01X01, P105 USB_A

Commit message: Switch designs to the 4.0.7 symbol and footprint library.
Parts:
- P105: symbol USB_A-RESCUE-usbabrkout -> USB_A
Changed lines of the file:
@@
 EESchema Schematic File Version 2
-LIBS:usbabrkout-rescue
 LIBS:local
 LIBS:power
@@
 D-
 $Comp
-L USB_A-RESCUE-usbabrkout P105
+L USB_A P105
 U 1 1 5ADE9713
 P 6000 3400

Commit message: Cleanup update to breakout boards. Upload to OSHpark.
Parts:
- PTC101: footprint local:C_1206_HandSoldering -> local:R_1206_HandSoldering
Changed lines of the file:
@@
 F 0 "PTC101" V 5150 3800 50  0000 C CNN
 F 1 "750mA" V 4950 3800 50  0000 C CNN
-F 2 "local:C_1206_HandSoldering" V 4980 3800 30  0001 C CNN
+F 2 "local:R_1206_HandSoldering" V 4980 3800 30  0001 C CNN
 F 3 "" V 5130 3800 30  0000 C CNN
 F 4 "6V" V 4880 3800 50  0000 C CNN "Voltage"

Commit message: Update USB-A breakout board to kicad 5.1. Regenerate output files.
Parts:
- P101, P102, P103, P104: symbol CONN_01X01 -> conn:CONN_01X01
- P105: symbol USB_A -> Local:USB_A
- PTC101: symbol PTC -> Local:PTC
Changed lines of the file:
@@
-EESchema Schematic File Version 2
-LIBS:local
-LIBS:power
-LIBS:device
-LIBS:transistors
-LIBS:conn
-LIBS:linear
-LIBS:regul
-LIBS:74xx
-LIBS:cmos4000
-LIBS:adc-dac
-LIBS:memory
-LIBS:xilinx
-LIBS:microcontrollers
-LIBS:dsp
-LIBS:microchip
-LIBS:analog_switches
-LIBS:motorola
-LIBS:texas
-LIBS:intel
-LIBS:audio
-LIBS:interface
-LIBS:digital-audio
-LIBS:philips
-LIBS:display
-LIBS:cypress
-LIBS:siliconi
-LIBS:opto
-LIBS:atmel
-LIBS:contrib
-LIBS:valves
-LIBS:usbabrkout-cache
-EELAYER 25 0
+EESchema Schematic File Version 4
+EELAYER 30 0
 EELAYER END
 $Descr A4 11693 8268
@@
 $EndDescr
 $Comp
-L CONN_01X01 P102
+L conn:CONN_01X01 P102
 U 1 1 5AD927DD
 P 4700 4000
@@
 $EndComp
 $Comp
-L CONN_01X01 P103
+L conn:CONN_01X01 P103
 U 1 1 5AD928A6
 P 4700 4200
@@
 $EndComp
 $Comp
-L GND #PWR01
+L power:GND #PWR01
 U 1 1 5AD92B85
 P 6400 4000
@@
 	6300 3300 6400 3300
 Wire Wire Line
-	6400 3300 6400 4000
+	6400 3300 6400 3800
 Wire Wire Line
 	4900 4200 6000 4200
@@
 D-
 $Comp
-L USB_A P105
+L Local:USB_A P105
 U 1 1 5ADE9713
 P 6000 3400
@@
 	5500 3800 5500 3500
 $Comp
-L VCC #PWR02
+L Local:VCC #PWR02
 U 1 1 5ADE9D9C
 P 5500 3500
@@
 $EndComp
 $Comp
-L CONN_01X01 P101
+L conn:CONN_01X01 P101
 U 1 1 5ADEA025
 P 4425 3800
@@
 $EndComp
 $Comp
-L CONN_01X01 P104
+L conn:CONN_01X01 P104
 U 1 1 5ADEA065
 P 4700 4400
@@
 Connection ~ 5500 3800
 $Comp
-L GND #PWR03
+L power:GND #PWR03
 U 1 1 5ADEA436
 P 5000 4500
@@
 	5000 4400 5000 4500
 Wire Wire Line
-	5200 3800 5800 3800
+	5200 3800 5500 3800
 Text Label 4650 3800 0    50   ~ 0
 +5v
 $Comp
-L PTC PTC101
+L Local:PTC PTC101
 U 1 1 5AE27E64
 P 5050 3800
@@
 	0    1    1    0
 $EndComp
+Wire Wire Line
+	6400 3800 6400 4000
+Wire Wire Line
+	5500 3800 5800 3800
 $EndSCHEMATC

Commit message: Fix rj45 break out board to point to 5.1 symbol libraries. Fix USB-A break out board to point to 5.1 symbol libraries. Fix USB-B break out board to point to 5.1 symbol libraries.
Parts:
- P101, P102, P103, P104: symbol conn:CONN_01X01 -> Connector_Generic:Conn_01x01
Changed lines of the file:
@@
 $EndDescr
 $Comp
-L conn:CONN_01X01 P102
+L Connector_Generic:Conn_01x01 P102
 U 1 1 5AD927DD
 P 4700 4000
@@
 $EndComp
 $Comp
-L conn:CONN_01X01 P103
+L Connector_Generic:Conn_01x01 P103
 U 1 1 5AD928A6
 P 4700 4200
@@
 $EndComp
 $Comp
-L conn:CONN_01X01 P101
+L Connector_Generic:Conn_01x01 P101
 U 1 1 5ADEA025
 P 4425 3800
@@
 $EndComp
 $Comp
-L conn:CONN_01X01 P104
+L Connector_Generic:Conn_01x01 P104
 U 1 1 5ADEA065
 P 4700 4400
