File: 8x16seg/8x16seg.sch (KiCad schematic (older format))
At the start: 48 parts, among them P1 CONN_01X08, P2 CONN_01X08, U1 TLC59282_REV, U2 TLC59282_REV, U3 TLC59282_REV, U4 TLC59282_REV, U5 TLC59282_REV, U6 TLC59282_REV, U7 TLC59282_REV, U8 TLC59282_REV, U9 TLC59282_REV

Commit message: Add NC to unused pins.
Connections:
- no-connect marks 0 -> 8
Changed lines of the file:
@@
 EESchema Schematic File Version 4
-LIBS:16seg-cache
 EELAYER 30 0
 EELAYER END
@@
 encoding utf-8
 Sheet 1 1
-Title "2 Digit 7-Segment Display"
-Date "2016-09-10"
-Rev "v1.2.0"
+Title "8 Digit 16-Segment Display"
+Date "2019-12-12"
+Rev "v1.0.0"
 Comp ""
 Comment1 ""
@@
 Wire Wire Line
 	8050 13450 8050 13600
+NoConn ~ 1200 7350
+NoConn ~ 3750 7350
+NoConn ~ 6300 7350
+NoConn ~ 8850 7350
+NoConn ~ 11400 7350
+NoConn ~ 13950 7350
+NoConn ~ 16500 7350
+NoConn ~ 19050 7350
 $EndSCHEMATC
